File: Projet 6 KICAD CLS COMPLET/Moteur1.kicad_sch (KiCad schematic)
At the start: 11 parts, among them SW2 SW_DIP_x02

Commit message: Projet 6 KICAD CLS COMPLET Correction
Parts:
- removed C8: 100n, symbol Device:C
- removed C9: 22n, symbol Device:C
- removed SW2: SW_DIP_x02, symbol Switch:SW_DIP_x02
- added C12, C13, C15, C22: 100n, symbol Device:C
- added C14: 100u, symbol Device:C_Polarized
- added C23: 22n, symbol Device:C
- added R15, R16: 10k, symbol Device:R
- R10, R11: value 150m -> 220m
Connections:
- net +3.3V: now also C15.1, R15.1, R16.1
- net GND: now also C12.2, C13.2, C14.2, C15.2
- net VCC: now also C12.1, C13.1, C14.1, C22.2
- net at U1.1 (CPO): now also C23.1
- net at U1.2 (CPI): now also C23.2
- net at R9.1, U1.26 (MS2): now also R15.2
- net at R8.1, U1.25 (MS1): now also R16.2
- net at U1.3 (VCP): now also C22.1
Other:
- note added: "Moteur TMC2225 1"
