File: Projet 6 KICAD CLS COMPLET Corrigé/LSM6DSOX.kicad_sch (KiCad schematic)
At the start: 6 parts, among them U3 LSM6DSOX

Commit message: Add files via upload
Parts:
- C1, C2: value 100nF -> 100n; footprint (none) -> Capacitor_SMD:C_0805_2012Metric
- R4, R5, R6: footprint (none) -> Resistor_SMD:R_0603_1608Metric
Changed lines of the file:
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@@
 			)
 		)
-		(property "Footprint" ""
+		(property "Footprint" "Resistor_SMD:R_0603_1608Metric"
 			(at 99.06 77.47 0)
 			(effects
@@
 			)
 		)
-		(property "Value" "100nF"
+		(property "Value" "100n"
 			(at 187.96 82.5562 0)
 			(effects
@@
 			)
 		)
-		(property "Footprint" ""
+		(property "Footprint" "Capacitor_SMD:C_0805_2012Metric"
 			(at 185.42 81.28 0)
 			(effects
@@
 			)
 		)
-		(property "Footprint" ""
+		(property "Footprint" "Resistor_SMD:R_0603_1608Metric"
 			(at 115.57 77.47 0)
 			(effects
@@
 			)
 		)
-		(property "Value" "100nF"
+		(property "Value" "100n"
 			(at 176.53 81.2863 90)
 			(effects
@@
 			)
 		)
-		(property "Footprint" ""
+		(property "Footprint" "Capacitor_SMD:C_0805_2012Metric"
 			(at 172.72 81.28 0)
 			(effects
@@
 			)
 		)
-		(property "Footprint" ""
+		(property "Footprint" "Resistor_SMD:R_0603_1608Metric"
 			(at 106.68 77.47 0)
 			(effects
