File: Projet 6 KICAD CLS COMPLET V3/Projet 6 KICAD CLS COMPLET.kicad_pcb (KiCad board)
At the start: 4 copper layers, 65 x 30 mm, 54 parts, among them J1 Raspberry Pi Zero 2w, J2 Conn_01x06, J3 Screw_Terminal_01x04, J4 Screw_Terminal_01x04, J5 Battery, U3 LSM6DSOX

Commit message: Add files via upload
Parts:
- C1, C12, C13, C15, C18, C2, C22, C23, C4, C5, C6, C7, C8, C9: footprint Capacitor_SMD:C_0805_2012Metric -> Capacitor_SMD:C_0603_1608Metric
- C11, C3: value 100n -> 2u2; footprint Capacitor_SMD:C_0805_2012Metric -> Capacitor_SMD:C_0603_1608Metric
- D3, D4: value LED -> GREEN LED
