File: Projet 6 KICAD CLS COMPLET V3/Projet 6 KICAD CLS COMPLET.kicad_sch (KiCad schematic)
At the start: 16 parts, among them J1 Raspberry Pi Zero 2w, J2 Conn_01x06, J3 Screw_Terminal_01x04, J4 Screw_Terminal_01x04, J5 Battery

Commit message: Add files via upload
Parts:
- C18, C4: footprint Capacitor_SMD:C_0805_2012Metric -> Capacitor_SMD:C_0603_1608Metric; MPN (none) -> 885012206071
- D3, D4: value LED -> GREEN LED; MPN (none) -> 150060GS55040
Changed lines of the file:
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@@
 		(on_board yes)
 		(dnp no)
-		(fields_autoplaced yes)
 		(property "Reference" "D4"
 			(at 105.41 174.3074 90)
@@
 			)
 		)
-		(property "Value" "LED"
-			(at 105.41 176.8474 90)
+		(property "Value" "GREEN LED"
+			(at 98.298 168.91 0)
 			(effects
 				(font
@@
 			)
 		)
+		(property "MPN" "150060GS55040"
+			(at 101.6 173.99 90)
+			(effects
+				(font
+					(size 1.27 1.27)
+				)
+				(hide yes)
+			)
+		)
 		(pin "2"
 		)
@@
 			)
 		)
-		(property "Footprint" "Capacitor_SMD:C_0805_2012Metric"
+		(property "Footprint" "Capacitor_SMD:C_0603_1608Metric"
 			(at 40.64 125.73 0)
 			(effects
@@
 			)
 		)
+		(property "MPN" "885012206071"
+			(at 40.64 125.73 90)
+			(effects
+				(font
+					(size 1.27 1.27)
+				)
+				(hide yes)
+			)
+		)
 		(pin "1"
 		)
@@
 			)
 		)
-		(property "Footprint" "Capacitor_SMD:C_0805_2012Metric"
+		(property "Footprint" "Capacitor_SMD:C_0603_1608Metric"
 			(at 57.15 170.18 0)
 			(effects
@@
 		)
 		(property "Description" "Unpolarized capacitor, small symbol"
+			(at 57.15 170.18 0)
+			(effects
+				(font
+					(size 1.27 1.27)
+				)
+				(hide yes)
+			)
+		)
+		(property "MPN" "885012206071"
 			(at 57.15 170.18 0)
 			(effects
@@
 		(on_board yes)
 		(dnp no)
-		(fields_autoplaced yes)
 		(property "Reference" "D3"
 			(at 92.71 174.3074 90)
@@
 			)
 		)
-		(property "Value" "LED"
-			(at 92.71 176.8474 90)
+		(property "Value" "GREEN LED"
+			(at 84.836 167.386 0)
 			(effects
 				(font
@@
 			(effects
 				(font
+					(size 1.27 1.27)
+				)
+				(hide yes)
+			)
+		)
+		(property "MPN" "150060GS55040"
+			(at 88.9 173.99 90)
+			(effects
+				(font
